File: kicad/DEV-G2-NANO.kicad_pcb (KiCad board)
At the start: 6 copper layers, 76.2 x 20.3 mm, 141 parts, among them J1 Lower Bank, J2 Upper Bank, J3 USB C, J4 HIC SWD, J5 RTC Battery, SW1 PTS815, U1 MIMXRT1171DVMAB, U10 TPS62825, U2 MAYA-W166-00B, U3 LSM6DSV, U4 LIS2MDL, U5 RTMC-G2-4IQ48, U6 W25Q64JWUUIQ, U7 MKL26Z128VFM4, U8 LM66200, U9 TPS62086, Y1 8MHz, Y2 16MHz, Y3 24MHz, Y4 32.768kHz

Commit message: moved wifi module from uSDHC2 to uSDHC1
Parts:
- moved R15 10.0 mm to (154.5, 83.1), turned to 180 degrees
- moved C41 1.33 mm to (156.7, 83.4)
- moved R18 1.17 mm to (164.0, 83.4), turned to 90 degrees
- moved R13 0.47 mm to (164.8, 83.4), turned to 90 degrees
- moved C5 0.16 mm to (172.7, 93.9)
Connections:
- U1 pad A4: Net-(U1C-GPIO_DISP_B2_15) -> (no net)
- U1 pad A7: Net-(U1C-GPIO_DISP_B2_14) -> Net-(U2A-WLAN_RESET)
- U1 pad B15: (no net) -> Net-(U1C-GPIO_SD_B1_04)
- U1 pad B3: (no net) -> Net-(U1C-GPIO_EMC_B1_17)
- U1 pad B4: (no net) -> Net-(U1C-GPIO_EMC_B1_18)
- U1 pad B5: (no net) -> Net-(U1C-GPIO_DISP_B2_08)
- U1 pad C4: (no net) -> Net-(U1C-GPIO_EMC_B1_19)
- U1 pad C5: (no net) -> Net-(U1C-GPIO_EMC_B1_12)
- U1 pad D15: (no net) -> Net-(U1C-GPIO_SD_B1_01)
- U1 pad E14: Net-(U1C-GPIO_SD_B2_05) -> unconnected-(U1C-GPIO_SD_B2_05-PadE14)
- U1 pad E15: Net-(U1C-GPIO_SD_B2_03) -> (no net)
- U1 pad F14: Net-(U1C-GPIO_SD_B2_04) -> (no net)
- U1 pad H13: Net-(U1C-GPIO_SD_B2_02) -> (no net)
- U1 pad J14: Net-(U1C-GPIO_SD_B2_01) -> (no net)
- U1 pad J15: Net-(U1C-GPIO_SD_B2_00) -> (no net)
- U1 pad M2: (no net) -> FAULT_IN
- U1 pad N3: (no net) -> FAULT_OUT
- U1 pad P2: (no net) -> UPDATE
- U2 pad A3: Net-(U1C-GPIO_SD_B2_02) -> Net-(U1C-GPIO_SD_B1_03)
- U2 pad A4: Net-(U1C-GPIO_SD_B2_04) -> Net-(U1C-GPIO_SD_B1_01)
- U2 pad A5: Net-(U1C-GPIO_SD_B2_00) -> Net-(U1C-GPIO_SD_B1_05)
- U2 pad B3: Net-(U1C-GPIO_SD_B2_03) -> Net-(U1C-GPIO_SD_B1_02)
- U2 pad B4: Net-(U1C-GPIO_SD_B2_05) -> Net-(U1C-GPIO_SD_B1_00)
- U2 pad B5: Net-(U1C-GPIO_SD_B2_01) -> Net-(U1C-GPIO_SD_B1_04)
- U2 pad E7: Net-(U1C-GPIO_SD_B1_00) -> Net-(U1C-GPIO_EMC_B1_12)
- U2 pad F7: Net-(U1C-GPIO_SD_B1_03) -> Net-(U1C-GPIO_EMC_B1_19)
- U2 pad H7: Net-(U1C-GPIO_SD_B1_02) -> Net-(U2A-WLAN_RESET)
- U2 pad J7: Net-(U1C-GPIO_SD_B1_05) -> Net-(U1C-GPIO_DISP_B2_08)
- U2 pad J8: Net-(U1C-GPIO_DISP_B2_15) -> Net-(U1C-GPIO_EMC_B1_18)
- U2 pad J9: Net-(U1C-GPIO_DISP_B2_14) -> Net-(U1C-GPIO_EMC_B1_17)
Routing:
- net Net-(U1C-GPIO_EMC_B1_19): track 0.00 -> 33.6 mm, vias 0 -> 2
- net Net-(U1C-GPIO_EMC_B1_12): track 0.00 -> 30.7 mm, vias 0 -> 2
- net Net-(U1C-GPIO_DISP_B2_15): track 30.7 -> 0.00 mm
- net Net-(U1C-GPIO_EMC_B1_17): track 0.00 -> 30.3 mm, vias 0 -> 2
- net Net-(U1C-GPIO_EMC_B1_18): track 0.00 -> 29.8 mm, vias 0 -> 2
- net FAULT_IN: track 8.05 -> 37.6 mm, vias 0 -> 2
- net Net-(U1C-GPIO_DISP_B2_08): track 0.00 -> 29.3 mm, vias 0 -> 2
- net FAULT_OUT: track 13.9 -> 42.3 mm, vias 0 -> 2
- net Net-(U1C-GPIO_DISP_B2_14): track 26.5 -> 0.00 mm
- net Net-(U2A-WLAN_RESET): track 0.00 -> 26.4 mm, vias 0 -> 2
- net UPDATE: track 13.3 -> 34.4 mm, vias 0 -> 2
- net Net-(U1C-GPIO_SD_B2_01): track 16.7 -> 0.00 mm, vias 2 -> 0
- net Net-(U1C-GPIO_SD_B1_04): track 0.00 -> 15.9 mm, vias 0 -> 2
- net Net-(U1C-GPIO_SD_B2_00): track 15.7 -> 0.00 mm, vias 2 -> 0
- net Net-(U1C-GPIO_SD_B2_05): track 14.0 -> 0.00 mm, vias 2 -> 0
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